File: light sensor basic.brd (EAGLE design)
At the start: 83.2 x 57.8 mm, 1 part

Commit message: test
Parts:
- added R1, R2: (no value), rcl:R1206
Changed lines of the file:
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@@
 <elements>
 <element name="U$1" library="voltera_community_lib" package="2X3_BOARD_V2" value="2X3_BOARD_V2" x="0" y="0" smashed="yes"/>
+<element name="R1" library="rcl" library_urn="urn:adsk.eagle:library:334" package="R1206" package3d_urn="urn:adsk.eagle:package:23540/2" value="" x="-8.255" y="-9.525" smashed="yes">
+<attribute name="NAME" x="-9.525" y="-8.255" size="1.27" layer="25"/>
+<attribute name="POPULARITY" value="19" x="-8.255" y="-9.525" size="1.778" layer="27" display="off"/>
+<attribute name="SPICEPREFIX" value="R" x="-8.255" y="-9.525" size="1.778" layer="27" display="off"/>
+<attribute name="VALUE" x="-9.525" y="-12.065" size="1.27" layer="27"/>
+</element>
+<element name="R2" library="rcl" library_urn="urn:adsk.eagle:library:334" package="R1206" package3d_urn="urn:adsk.eagle:package:23540/2" value="" x="-8.255" y="-13.97" smashed="yes">
+<attribute name="NAME" x="-9.525" y="-12.7" size="1.27" layer="25"/>
+<attribute name="POPULARITY" value="19" x="-8.255" y="-13.97" size="1.778" layer="27" display="off"/>
+<attribute name="SPICEPREFIX" value="R" x="-8.255" y="-13.97" size="1.778" layer="27" display="off"/>
+<attribute name="VALUE" x="-9.525" y="-16.51" size="1.27" layer="27"/>
+</element>
 </elements>
 <signals>
@@
 </board>
 </drawing>
+<compatibility>
+<note version="8.2" severity="warning">
+Since Version 8.2, EAGLE supports online libraries. The ids
+of those online libraries will not be understood (or retained)
+with this version.
+</note>
+<note version="8.3" severity="warning">
+Since Version 8.3, EAGLE supports URNs for individual library
+assets (packages, symbols, and devices). The URNs of those assets
+will not be understood (or retained) with this version.
+</note>
+<note version="8.3" severity="warning">
+Since Version 8.3, EAGLE supports the association of 3D packages
+with devices in libraries, schematics, and board files. Those 3D
+packages will not be understood (or retained) with this version.
+</note>
+</compatibility>
 </eagle>

Commit message: new test
Parts:
- removed R1, R2: (no value), rcl:R1206
Changed lines of the file:
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@@
 <elements>
 <element name="U$1" library="voltera_community_lib" package="2X3_BOARD_V2" value="2X3_BOARD_V2" x="0" y="0" smashed="yes"/>
-<element name="R1" library="rcl" library_urn="urn:adsk.eagle:library:334" package="R1206" package3d_urn="urn:adsk.eagle:package:23540/2" value="" x="-8.255" y="-9.525" smashed="yes">
-<attribute name="NAME" x="-9.525" y="-8.255" size="1.27" layer="25"/>
-<attribute name="POPULARITY" value="19" x="-8.255" y="-9.525" size="1.778" layer="27" display="off"/>
-<attribute name="SPICEPREFIX" value="R" x="-8.255" y="-9.525" size="1.778" layer="27" display="off"/>
-<attribute name="VALUE" x="-9.525" y="-12.065" size="1.27" layer="27"/>
-</element>
-<element name="R2" library="rcl" library_urn="urn:adsk.eagle:library:334" package="R1206" package3d_urn="urn:adsk.eagle:package:23540/2" value="" x="-8.255" y="-13.97" smashed="yes">
-<attribute name="NAME" x="-9.525" y="-12.7" size="1.27" layer="25"/>
-<attribute name="POPULARITY" value="19" x="-8.255" y="-13.97" size="1.778" layer="27" display="off"/>
-<attribute name="SPICEPREFIX" value="R" x="-8.255" y="-13.97" size="1.778" layer="27" display="off"/>
-<attribute name="VALUE" x="-9.525" y="-16.51" size="1.27" layer="27"/>
-</element>
 </elements>
 <signals>
@@
 </board>
 </drawing>
-<compatibility>
-<note version="8.2" severity="warning">
-Since Version 8.2, EAGLE supports online libraries. The ids
-of those online libraries will not be understood (or retained)
-with this version.
-</note>
-<note version="8.3" severity="warning">
-Since Version 8.3, EAGLE supports URNs for individual library
-assets (packages, symbols, and devices). The URNs of those assets
-will not be understood (or retained) with this version.
-</note>
-<note version="8.3" severity="warning">
-Since Version 8.3, EAGLE supports the association of 3D packages
-with devices in libraries, schematics, and board files. Those 3D
-packages will not be understood (or retained) with this version.
-</note>
-</compatibility>
 </eagle>

Commit message: try againx2
Parts:
- added U1: VCNT2020, VCNT2020:XDCR_VCNT2020
Changed lines of the file:
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@@
 <elements>
 <element name="U$1" library="voltera_community_lib" package="2X3_BOARD_V2" value="2X3_BOARD_V2" x="0" y="0" smashed="yes"/>
+<element name="U1" library="VCNT2020" package="XDCR_VCNT2020" value="VCNT2020" x="-7.62" y="-10.16" smashed="yes">
+<attribute name="CHECK_PRICES" value="https://www.snapeda.com/parts/VCNT2020/Vishay+Semiconductor+Opto+Division/view-part/?ref=eda" x="-7.62" y="-10.16" size="1.778" layer="27" display="off"/>
+<attribute name="DESCRIPTION" value="                                                      Reflective Optical Sensor 0.02 (0.5mm) 4-SMD Module                                              " x="-7.62" y="-10.16" size="1.778" layer="27" display="off"/>
+<attribute name="DIGIKEY_PART_NUMBER" value="VCNT2020TR-ND" x="-7.62" y="-10.16" size="1.778" layer="27" display="off"/>
+<attribute name="MF" value="Vishay" x="-7.62" y="-10.16" size="1.778" layer="27" display="off"/>
+<attribute name="MP" value="VCNT2020" x="-7.62" y="-10.16" size="1.778" layer="27" display="off"/>
+<attribute name="NAME" x="-10.16" y="-8.128" size="1.27" layer="25"/>
+<attribute name="PACKAGE" value="None" x="-7.62" y="-10.16" size="1.778" layer="27" display="off"/>
+<attribute name="SNAPEDA_LINK" value="https://www.snapeda.com/parts/VCNT2020/Vishay+Semiconductor+Opto+Division/view-part/?ref=snap" x="-7.62" y="-10.16" size="1.778" layer="27" display="off"/>
+<attribute name="VALUE" x="-10.16" y="-13.462" size="1.27" layer="27"/>
+</element>
 </elements>
 <signals>

Commit message: wont change
github schematic absolutely refuses to update
Parts:
- added R1: (no value), rcl:R1206
Changed lines of the file:
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@@
 <drawing>
 <settings>
-<setting alwaysvectorfont="no"/>
+<setting alwaysvectorfont="yes"/>
 <setting verticaltext="up"/>
 </settings>
@@
 <attribute name="VALUE" x="-10.16" y="-13.462" size="1.27" layer="27"/>
 </element>
+<element name="R1" library="rcl" library_urn="urn:adsk.eagle:library:334" package="R1206" package3d_urn="urn:adsk.eagle:package:23540/2" value="" x="-8.255" y="-17.145" smashed="yes">
+<attribute name="NAME" x="-9.525" y="-15.875" size="1.27" layer="25"/>
+<attribute name="POPULARITY" value="19" x="-8.255" y="-17.145" size="1.778" layer="27" display="off"/>
+<attribute name="SPICEPREFIX" value="R" x="-8.255" y="-17.145" size="1.778" layer="27" display="off"/>
+<attribute name="VALUE" x="-9.525" y="-19.685" size="1.27" layer="27"/>
+</element>
 </elements>
 <signals>
@@
 </board>
 </drawing>
+<compatibility>
+<note version="8.2" severity="warning">
+Since Version 8.2, EAGLE supports online libraries. The ids
+of those online libraries will not be understood (or retained)
+with this version.
+</note>
+<note version="8.3" severity="warning">
+Since Version 8.3, EAGLE supports URNs for individual library
+assets (packages, symbols, and devices). The URNs of those assets
+will not be understood (or retained) with this version.
+</note>
+<note version="8.3" severity="warning">
+Since Version 8.3, EAGLE supports the association of 3D packages
+with devices in libraries, schematics, and board files. Those 3D
+packages will not be understood (or retained) with this version.
+</note>
+</compatibility>
 </eagle>

Commit message: SHOULD WORK
Parts:
- added C1: 0.1uF, rcl:C1206
- added J1: UJ2-MIBH-G-SMT-TR, UJ2-MIBH-G-SMT-TR:CUI_UJ2-MIBH-G-SMT-TR
- added LED1: (no value), led:SML0805
- added R2: TC33X-2-203E, TC33X-2-203E:TRIM_TC33X-2-203E
- added R3: 150, rcl:R0805
- added T1: (no value), transistor:SOT23-EBC
- added TP1, TP2, TP3, TP4: (no value), rcl:R1206
- R1: value (none) -> 82; device rcl:R1206 -> rcl:R0805
- moved R1 70.0 mm to (41.3, 32.4)
- moved U1 56.2 mm to (29.8, 31.8)
Connections:
- new net GND: C1.1, J1.5, J1.S1, J1.S2, J1.S3, J1.S4, R2.3, T1.E, TP4.1, TP4.2, U1.4
- new net N$1: R1.1, U1.3
- new net N$2: R2.1, TP1.1, TP1.2, U1.1
- new net N$3: R2.2, T1.B, TP2.1, TP2.2
- new net N$4: LED1.C, T1.C
- new net VCC: C1.2, J1.1, R1.2, R3.1, TP3.1, TP3.2, U1.2

Commit message: c
Parts:
- R1: device rcl:R0805 -> rcl:R1206
Changed lines of the file:
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@@
 <drawing>
 <settings>
-<setting alwaysvectorfont="yes"/>
+<setting alwaysvectorfont="no"/>
 <setting verticaltext="up"/>
 </settings>
@@
 <attribute name="VALUE" x="27.305" y="28.448" size="1.27" layer="27"/>
 </element>
-<element name="R1" library="rcl" library_urn="urn:adsk.eagle:library:334" package="R0805" package3d_urn="urn:adsk.eagle:package:23553/2" value="82" x="41.275" y="32.385" smashed="yes">
+<element name="R1" library="rcl" library_urn="urn:adsk.eagle:library:334" package="R1206" package3d_urn="urn:adsk.eagle:package:23540/2" value="82" x="41.275" y="32.385" smashed="yes">
 <attribute name="NAME" x="40.64" y="33.655" size="1.27" layer="25"/>
-<attribute name="POPULARITY" value="85" x="41.275" y="32.385" size="1.778" layer="27" display="off"/>
+<attribute name="POPULARITY" value="19" x="41.275" y="32.385" size="1.778" layer="27" display="off"/>
 <attribute name="SPICEPREFIX" value="R" x="41.275" y="32.385" size="1.778" layer="27" display="off"/>
 <attribute name="VALUE" x="40.64" y="29.845" size="1.27" layer="27"/>
@@
 <contactref element="U1" pad="3"/>
 <contactref element="R1" pad="1"/>
-<wire x1="40.325" y1="32.385" x2="30.475" y2="32.475" width="0" layer="19" extent="1-1"/>
+<wire x1="30.475" y1="32.475" x2="39.853" y2="32.385" width="0" layer="19" extent="1-1"/>
 </signal>
 <signal name="VCC">
@@
 <contactref element="TP3" pad="1"/>
 <contactref element="TP3" pad="2"/>
-<wire x1="16.027" y1="17.145" x2="13.183" y2="17.145" width="0" layer="19" extent="1-1"/>
-<wire x1="15.845" y1="26.17" x2="16.027" y2="17.145" width="0" layer="19" extent="1-1"/>
+<wire x1="29.275" y1="31.125" x2="42.697" y2="32.385" width="0" layer="19" extent="1-1"/>
+<wire x1="15.845" y1="26.17" x2="29.275" y2="31.125" width="0" layer="19" extent="1-1"/>
 <wire x1="13.02" y1="33.655" x2="15.845" y2="26.17" width="0" layer="19" extent="1-1"/>
+<wire x1="16.027" y1="17.145" x2="15.845" y2="26.17" width="0" layer="19" extent="1-1"/>
+<wire x1="13.183" y1="17.145" x2="16.027" y2="17.145" width="0" layer="19" extent="1-1"/>
 <wire x1="23.625" y1="50.165" x2="13.02" y2="33.655" width="0" layer="19" extent="1-1"/>
-<wire x1="42.225" y1="32.385" x2="23.625" y2="50.165" width="0" layer="19" extent="1-1"/>
-<wire x1="29.275" y1="31.125" x2="42.225" y2="32.385" width="0" layer="19" extent="1-1"/>
 </signal>
 <signal name="GND">

Commit message: a
Parts:
- moved J1 50.6 mm to (61.6, 47.6)
- moved LED1 7.96 mm to (6.99, 34.3)
Changed lines of the file:
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@@
 <attribute name="VALUE" x="12.065" y="40.005" size="1.27" layer="27"/>
 </element>
-<element name="LED1" library="led" library_urn="urn:adsk.eagle:library:259" package="SML0805" package3d_urn="urn:adsk.eagle:package:15830/1" value="" x="13.97" y="38.1" smashed="yes">
-<attribute name="NAME" x="12.47" y="39.1" size="1.27" layer="25"/>
-<attribute name="POPULARITY" value="17" x="13.97" y="38.1" size="1.778" layer="27" display="off"/>
-<attribute name="VALUE" x="12.47" y="36.1" size="1.27" layer="27"/>
+<element name="LED1" library="led" library_urn="urn:adsk.eagle:library:259" package="SML0805" package3d_urn="urn:adsk.eagle:package:15830/1" value="" x="6.985" y="34.29" smashed="yes">
+<attribute name="NAME" x="5.485" y="35.29" size="1.27" layer="25"/>
+<attribute name="POPULARITY" value="17" x="6.985" y="34.29" size="1.778" layer="27" display="off"/>
+<attribute name="VALUE" x="5.485" y="32.29" size="1.27" layer="27"/>
 </element>
 <element name="R3" library="rcl" library_urn="urn:adsk.eagle:library:334" package="R0805" package3d_urn="urn:adsk.eagle:package:23553/2" value="150" x="13.97" y="33.655" smashed="yes">
@@
 <attribute name="VALUE" x="13.335" y="31.115" size="1.27" layer="27"/>
 </element>
-<element name="J1" library="UJ2-MIBH-G-SMT-TR" package="CUI_UJ2-MIBH-G-SMT-TR" value="UJ2-MIBH-G-SMT-TR" x="17.145" y="23.495" smashed="yes">
-<attribute name="MANUFACTURER" value="CUI" x="17.145" y="23.495" size="1.778" layer="27" display="off"/>
-<attribute name="MAXIMUM_PACKAGE_HEIGHT" value="2.95 mm" x="17.145" y="23.495" size="1.778" layer="27" display="off"/>
-<attribute name="NAME" x="13.145" y="28.595" size="1.27" layer="25"/>
-<attribute name="PARTREV" value="1.0" x="17.145" y="23.495" size="1.778" layer="27" display="off"/>
-<attribute name="STANDARD" value="Manufacturer Recommendations" x="17.145" y="23.495" size="1.778" layer="27" display="off"/>
-<attribute name="VALUE" x="13.145" y="27.195" size="1.27" layer="27"/>
+<element name="J1" library="UJ2-MIBH-G-SMT-TR" package="CUI_UJ2-MIBH-G-SMT-TR" value="UJ2-MIBH-G-SMT-TR" x="61.595" y="47.625" smashed="yes">
+<attribute name="MANUFACTURER" value="CUI" x="61.595" y="47.625" size="1.778" layer="27" display="off"/>
+<attribute name="MAXIMUM_PACKAGE_HEIGHT" value="2.95 mm" x="61.595" y="47.625" size="1.778" layer="27" display="off"/>
+<attribute name="NAME" x="57.595" y="52.725" size="1.27" layer="25"/>
+<attribute name="PARTREV" value="1.0" x="61.595" y="47.625" size="1.778" layer="27" display="off"/>
+<attribute name="STANDARD" value="Manufacturer Recommendations" x="61.595" y="47.625" size="1.778" layer="27" display="off"/>
+<attribute name="VALUE" x="57.595" y="51.325" size="1.27" layer="27"/>
 </element>
 <element name="TP3" library="rcl" library_urn="urn:adsk.eagle:library:334" package="R1206" package3d_urn="urn:adsk.eagle:package:23540/2" value="" x="14.605" y="17.145" smashed="yes">
@@
 <contactref element="TP3" pad="2"/>
 <wire x1="29.275" y1="31.125" x2="42.697" y2="32.385" width="0" layer="19" extent="1-1"/>
-<wire x1="15.845" y1="26.17" x2="29.275" y2="31.125" width="0" layer="19" extent="1-1"/>
-<wire x1="13.02" y1="33.655" x2="15.845" y2="26.17" width="0" layer="19" extent="1-1"/>
-<wire x1="16.027" y1="17.145" x2="15.845" y2="26.17" width="0" layer="19" extent="1-1"/>
+<wire x1="60.295" y1="50.3" x2="29.275" y2="31.125" width="0" layer="19" extent="1-1"/>
+<wire x1="13.02" y1="33.655" x2="60.295" y2="50.3" width="0" layer="19" extent="1-1"/>
+<wire x1="16.027" y1="17.145" x2="60.295" y2="50.3" width="0" layer="19" extent="1-1"/>
 <wire x1="13.183" y1="17.145" x2="16.027" y2="17.145" width="0" layer="19" extent="1-1"/>
 <wire x1="23.625" y1="50.165" x2="13.02" y2="33.655" width="0" layer="19" extent="1-1"/>
@@
 <contactref element="TP4" pad="2"/>
 <wire x1="16.027" y1="12.7" x2="13.183" y2="12.7" width="0" layer="19" extent="1-1"/>
-<wire x1="13.195" y1="23.495" x2="13.183" y2="12.7" width="0" layer="19" extent="1-1"/>
-<wire x1="15.945" y1="23.495" x2="13.195" y2="23.495" width="0" layer="19" extent="1-1"/>
-<wire x1="18.345" y1="23.495" x2="15.945" y2="23.495" width="0" layer="19" extent="1-1"/>
-<wire x1="18.445" y1="26.17" x2="18.345" y2="23.495" width="0" layer="19" extent="1-1"/>
-<wire x1="21.095" y1="23.495" x2="18.345" y2="23.495" width="0" layer="19" extent="1-1"/>
-<wire x1="13.02" y1="42.08" x2="18.445" y2="26.17" width="0" layer="19" extent="1-1"/>
+<wire x1="57.645" y1="47.625" x2="13.183" y2="12.7" width="0" layer="19" extent="1-1"/>
+<wire x1="60.395" y1="47.625" x2="57.645" y2="47.625" width="0" layer="19" extent="1-1"/>
+<wire x1="62.795" y1="47.625" x2="60.395" y2="47.625" width="0" layer="19" extent="1-1"/>
+<wire x1="62.895" y1="50.3" x2="62.795" y2="47.625" width="0" layer="19" extent="1-1"/>
+<wire x1="65.545" y1="47.625" x2="62.795" y2="47.625" width="0" layer="19" extent="1-1"/>
+<wire x1="13.02" y1="42.08" x2="62.895" y2="50.3" width="0" layer="19" extent="1-1"/>
 <wire x1="13.44" y1="50.435" x2="13.02" y2="42.08" width="0" layer="19" extent="1-1"/>
 <wire x1="20.825" y1="50.165" x2="13.44" y2="50.435" width="0" layer="19" extent="1-1"/>
@@
 <contactref element="T1" pad="C"/>
 <contactref element="LED1" pad="C"/>
-<wire x1="13.97" y1="44.28" x2="12.92" y2="38.1" width="0" layer="19" extent="1-1"/>
+<wire x1="13.97" y1="44.28" x2="5.935" y2="34.29" width="0" layer="19" extent="1-1"/>
 </signal>
 </signals>
