File: light sensor basic.brd (EAGLE design)
At the start: 83.2 x 57.8 mm, 11 parts, among them U1 VCNT2020

Commit message: Add files via upload
Parts:
- added J1: UJ2-MIBH-G-SMT-TR, UJ2-MIBH-G-SMT-TR:CUI_UJ2-MIBH-G-SMT-TR
- added LED1: (no value), led:SML0805
- TP1: device rcl:R1206 -> rcl:R0805
- moved TP4 117.7 mm to (-102.9, 20.3)
- moved R1 116.8 mm to (-73.7, 53.3), turned to 90 degrees
- moved U1 112.0 mm to (-80.0, 53.3), turned to 270 degrees
- moved C1 107.4 mm to (-85.1, 53.3), turned to 90 degrees
- moved U$1 106.9 mm to (-106.7, 6.35)
- moved TP1 92.9 mm to (-69.8, 47.0), turned to 270 degrees
- moved R2 85.4 mm to (-64.8, 21.6), turned to 90 degrees
- moved TP3 82.1 mm to (-59.7, 52.1), turned to 270 degrees
- moved T1 75.2 mm to (-59.7, 27.9)
- moved TP2 75.1 mm to (-54.6, 33.0), turned to 270 degrees
- moved R3 74.4 mm to (-59.7, 44.5), turned to 90 degrees
Connections:
- removed net N$4 (its old number): T1.C
- new net N$12: LED1.A, R3.1
- new net N$2: J1.2, J1.3
- new net N$5: LED1.C, T1.C
- net GND: now also J1.5, J1.S1, J1.S2, J1.S3, J1.S4
- net VCC: now also J1.1, R3.2; no longer R3.1
Routing:
- net VCC: track 0.00 -> 56.6 mm
- net N$10: track 0.00 -> 45.7 mm
- net N$4: track 0.00 -> 21.6 mm
- net GND: track 0.00 -> 17.2 mm
- net N$12: track 0.00 -> 6.89 mm
- net N$1: track 0.00 -> 5.95 mm
- net N$5: track 0.00 -> 5.47 mm
- added copper zone on layer 1, net GND
Other:
- board size 83.2 x 57.8 mm -> 160 x 100 mm
- board text added: "C1"
- board text added: "K<-LED1"
- board text added: "R1"
- board text added: "R2"
- board text added: "R3"
- board text added: "T1"
- board text added: "TP1"
- board text added: "TP2"
- board text added: "TP3"
- board text added: "U1"
